File: Kicad/Keeb_small_symetrical_hotswap_left/Keeb.kicad_pcb (KiCad board)
At the start: 2 copper layers, 96.3 x 99.3 mm, 20 parts, among them J1 TYPE-C-31-M-12, SW1 CherryMX, SW10 CherryMX, SW11 CherryMX, SW13 CherryMX, SW14 CherryMX, SW15 CherryMX, SW16 CherryMX, SW17 CherryMX, SW18 CherryMX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

Commit message: done some routing
Connections:
- SW1 pad 1: 5 -> 27
- SW10 pad 1: 16 -> unconnected-(SW10-Pad1)
- SW11 pad 2: 15 -> unconnected-(SW11-Pad2)
- SW13 pad 2: 12 -> unconnected-(SW13-Pad2)
- SW14 pad 2: 13 -> unconnected-(SW14-Pad2)
- SW15 pad 2: 14 -> 20
- SW16 pad 1: 6 -> 26
- SW17 pad 1: 9 -> unconnected-(SW17-Pad1)
- SW18 pad 1: 10 -> unconnected-(SW18-Pad1)
- SW19 pad 1: 11 -> 21
- SW20 pad 1: 7 -> 22
- SW3 pad 2: 21 -> unconnected-(SW3-Pad2)
- SW4 pad 2: 22 -> unconnected-(SW4-Pad2)
- SW5 pad 2: 26 -> unconnected-(SW5-Pad2)
- SW6 pad 2: 18 -> unconnected-(SW6-Pad2)
- SW7 pad 2: 19 -> unconnected-(SW7-Pad2)
- SW8 pad 2: 20 -> unconnected-(SW8-Pad2)
- SW9 pad 1: 17 -> unconnected-(SW9-Pad1)
Routing:
- net 3v3: track 0.00 -> 175.0 mm
- net GND: track 0.00 -> 169.4 mm
- net VSYS: track 0.00 -> 104.4 mm
- net 1: track 0.00 -> 103.7 mm
- net 2: track 0.00 -> 96.6 mm
- net 21: track 0.00 -> 50.4 mm
- net 20: track 0.00 -> 49.4 mm
- net 22: track 0.00 -> 29.9 mm
- net 26: track 0.00 -> 20.7 mm
- net 27: track 0.00 -> 14.0 mm

Commit message: More or less MVP of left keabord PCB
Parts:
- moved J1 3.10 mm to (133.3, 36.0), turned to 180 degrees
Connections:
- SW10 pad 1: unconnected-(SW10-Pad1) -> 11
- SW11 pad 1: GND -> 12
- SW11 pad 2: unconnected-(SW11-Pad2) -> GND
- SW13 pad 2: unconnected-(SW13-Pad2) -> 19
- SW14 pad 2: unconnected-(SW14-Pad2) -> 18
- SW17 pad 1: unconnected-(SW17-Pad1) -> 16
- SW18 pad 1: unconnected-(SW18-Pad1) -> 17
- SW3 pad 2: unconnected-(SW3-Pad2) -> 7
- SW4 pad 2: unconnected-(SW4-Pad2) -> 6
- SW5 pad 2: unconnected-(SW5-Pad2) -> 5
- SW6 pad 2: unconnected-(SW6-Pad2) -> 9
- SW7 pad 2: unconnected-(SW7-Pad2) -> 8
- SW9 pad 1: unconnected-(SW9-Pad1) -> 10
Routing:
- net GND: track 169.4 -> 549.3 mm
- net 0: track 0.00 -> 148.5 mm
- net 16: track 0.00 -> 73.1 mm
- net 19: track 0.00 -> 73.1 mm
- net 9: track 0.00 -> 68.0 mm
- net 10: track 0.00 -> 59.9 mm
- net 17: track 0.00 -> 58.8 mm
- net 7: track 0.00 -> 55.9 mm
- net 18: track 0.00 -> 50.4 mm
- net 8: track 0.00 -> 48.2 mm
- net 11: track 0.00 -> 39.2 mm
- net 6: track 0.00 -> 37.2 mm
- net 5: track 0.00 -> 18.9 mm
- net 12: track 0.00 -> 17.5 mm
- net VSYS: track 104.4 -> 114.3 mm
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Other:
- outline, holes or cut-outs redrawn
