File: Kicad/Keeb_small_symetrical_hotswap_left/Keeb.kicad_pcb (KiCad board)
At the start: 2 copper layers, 96.3 x 99.3 mm, 20 parts, among them J1 TYPE-C-31-M-12, SW1 CherryMX, SW10 CherryMX, SW11 CherryMX, SW13 CherryMX, SW14 CherryMX, SW15 CherryMX, SW16 CherryMX, SW17 CherryMX, SW18 CherryMX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

Commit message: rm holes for controller
Parts:
- U1: footprint MCU_RaspberryPi_and_Boards:RPi_Pico_SMD_TH -> MCU_RaspberryPi_and_Boards:RPi_Pico_SMD_TH_NO_HOLES

Commit message: min
Parts:
- J1: footprint USB-C-Power-tester:TYPE-C-31-M-12 -> TypeC:HRO_TYPE-C-31-M-12

Commit message: Added mounting holes to the PCB
Parts:
- added H1: MountingHole, MountingHole:MountingHole_3.2mm_M3, F.Cu at (121.7, 46.1)
- added H2: MountingHole, MountingHole:MountingHole_3.2mm_M3, F.Cu at (159.8, 70.1)
- added H3: MountingHole, MountingHole:MountingHole_3.2mm_M3, F.Cu at (159.8, 51.0)
- added H4: MountingHole, MountingHole:MountingHole_3.2mm_M3, F.Cu at (178.8, 58.1)
- added H5: MountingHole, MountingHole:MountingHole_3.2mm_M3, F.Cu at (118.2, 104.4)
- added H7: MountingHole, MountingHole:MountingHole_3.2mm_M3, F.Cu at (121.7, 84.2)
- added H8: MountingHole, MountingHole:MountingHole_3.2mm_M3, F.Cu at (178.8, 96.2)
- added H9: MountingHole, MountingHole:MountingHole_3.2mm_M3, F.Cu at (151.2, 123.4)
Routing:
- net 11: track 57.7 -> 70.2 mm
- net VSYS: track 114.3 -> 125.7 mm
- net 2: track 104.5 -> 115.6 mm
- net 1: track 109.2 -> 120.3 mm
- net 9: track 68.0 -> 78.2 mm
- net 12: track 37.2 -> 47.3 mm
- net 6: track 37.2 -> 46.9 mm
- net GND: track 549.3 -> 556.0 mm
- net 8: track 48.2 -> 53.8 mm
- net 26: track 20.7 -> 25.9 mm
- net 21: track 50.4 -> 46.0 mm
- net 20: track 49.4 -> 45.3 mm
- net 5: track 18.9 -> 21.7 mm
- net 7: track 55.9 -> 58.6 mm
- net 18: track 50.4 -> 48.2 mm
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