File: Kicad/Keeb_small_symetrical_hotswap_left/Keeb.kicad_sch (KiCad schematic)
At the start: 20 parts, among them J1 TYPE-C-31-M-12, SW1 CherryMX, SW10 CherryMX, SW11 CherryMX, SW13 CherryMX, SW14 CherryMX, SW15 CherryMX, SW16 CherryMX, SW17 CherryMX, SW18 CherryMX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

Commit message: done some routing
Connections:
- net 10: no longer SW18.1
- net 11: no longer SW19.1
- net 12: no longer SW13.2
- net 13: no longer SW14.2
- net 14: no longer SW15.2
- net 15: no longer SW11.2
- net 16: no longer SW10.1
- net 17: no longer SW9.1
- net 18: no longer SW6.2
- net 19: no longer SW7.2
- net 20: now also SW15.2; no longer SW8.2
- net 21: now also SW19.1; no longer SW3.2
- net 22: now also SW20.1; no longer SW4.2
- net 26: now also SW16.1; no longer SW5.2
- net 27: now also SW1.1
- net 5: no longer SW1.1
- net 6: no longer SW16.1
- net 7: no longer SW20.1
- net 9: no longer SW17.1

Commit message: More or less MVP of left keabord PCB
Parts:
- J1: footprint TypeC:HRO_TYPE-C-31-M-12 -> USB-C-Power-tester:TYPE-C-31-M-12
Connections:
- net 10: now also SW9.1
- net 11: now also SW10.1
- net 12: now also SW11.1
- net 16: now also SW17.1
- net 17: now also SW18.1
- net 18: now also SW14.2
- net 19: now also SW13.2
- net 5: now also SW5.2
- net 6: now also SW4.2
- net 7: now also SW3.2
- net 8: now also SW7.2
- net 9: now also SW6.2
- net GND: now also SW11.2; no longer SW11.1
Changed lines of the file:
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@@
-    (stroke (width 0) (type default))
-  )
-  (wire (pts (xy 133.35 77.47) (xy 133.35 85.09))
     (stroke (width 0) (type default))
   )
@@
     (stroke (width 0) (type default))
   )
-  (wire (pts (xy 143.51 77.47) (xy 133.35 77.47))
-    (stroke (width 0) (type default))
-  )
   (wire (pts (xy 120.65 72.39) (xy 120.65 85.09))
     (stroke (width 0) (type default))
@@
     (stroke (width 0) (type default))
   )
-  (wire (pts (xy 143.51 72.39) (xy 143.51 77.47))
+  (wire (pts (xy 143.51 72.39) (xy 143.51 85.09))
     (stroke (width 0) (type default))
   )
@@
     )
   )
+  (global_label "11" (shape input) (at 133.35 72.39 270) (fields_autoplaced)
+    (effects (font (size 1.27 1.27)) (justify right))
+    (property "Intersheetrefs" "${INTERSHEET_REFS}" (at 133.35 77.14 90)
+      (effects (font (size 1.27 1.27)) (justify right) hide)
+    )
+  )
   (global_label "5" (shape input) (at 49.53 96.52 180) (fields_autoplaced)
     (effects (font (size 1.27 1.27)) (justify right))
@@
     )
   )
+  (global_label "8" (shape input) (at 130.81 72.39 270) (fields_autoplaced)
+    (effects (font (size 1.27 1.27)) (justify right))
+    (property "Intersheetrefs" "${INTERSHEET_REFS}" (at 130.81 75.9305 90)
+      (effects (font (size 1.27 1.27)) (justify right) hide)
+    )
+  )
   (global_label "2" (shape input) (at 91.44 36.83 0) (fields_autoplaced)
     (effects (font (size 1.27 1.27)) (justify left))
@@
     )
   )
+  (global_label "9" (shape input) (at 130.81 62.23 270) (fields_autoplaced)
+    (effects (font (size 1.27 1.27)) (justify right))
+    (property "Intersheetrefs" "${INTERSHEET_REFS}" (at 130.81 65.7705 90)
+      (effects (font (size 1.27 1.27)) (justify right) hide)
+    )
+  )
   (global_label "14" (shape input) (at 49.53 127 180) (fields_autoplaced)
     (effects (font (size 1.27 1.27)) (justify right))
@@
     )
   )
-  (global_label "GND" (shape input) (at 133.35 85.09 270) (fields_autoplaced)
-    (effects (font (size 1.27 1.27)) (justify right))
-    (property "Intersheetrefs" "${INTERSHEET_REFS}" (at 133.35 91.2915 90)
-      (effects (font (size 1.27 1.27)) (justify right) hide)
-    )
-  )
   (global_label "3v3" (shape input) (at 87.63 29.21 0) (fields_autoplaced)
     (effects (font (size 1.27 1.27)) (justify left))
@@
     )
   )
+  (global_label "19" (shape input) (at 156.21 62.23 270) (fields_autoplaced)
+    (effects (font (size 1.27 1.27)) (justify right))
+    (property "Intersheetrefs" "${INTERSHEET_REFS}" (at 156.21 66.98 90)
+      (effects (font (size 1.27 1.27)) (justify right) hide)
+    )
+  )
   (global_label "9" (shape input) (at 49.53 109.22 180) (fields_autoplaced)
     (effects (font (size 1.27 1.27)) (justify right))
@@
     )
   )
+  (global_label "16" (shape input) (at 158.75 62.23 270) (fields_autoplaced)
+    (effects (font (size 1.27 1.27)) (justify right))
+    (property "Intersheetrefs" "${INTERSHEET_REFS}" (at 158.75 66.98 90)
+      (effects (font (size 1.27 1.27)) (justify right) hide)
+    )
+  )
   (global_label "VSYS" (shape input) (at 99.06 34.29 0) (fields_autoplaced)
     (effects (font (size 1.27 1.27)) (justify left))
@@
     )
   )
+  (global_label "6" (shape input) (at 118.11 72.39 270) (fields_autoplaced)
+    (effects (font (size 1.27 1.27)) (justify right))
+    (property "Intersheetrefs" "${INTERSHEET_REFS}" (at 118.11 75.9305 90)
+      (effects (font (size 1.27 1.27)) (justify right) hide)
+    )
+  )
   (global_label "0" (shape input) (at 49.53 81.28 180) (fields_autoplaced)
     (effects (font (size 1.27 1.27)) (justify right))
@@
     )
   )
+  (global_label "12" (shape input) (at 133.35 85.09 270) (fields_autoplaced)
+    (effects (font (size 1.27 1.27)) (justify right))
+    (property "Intersheetrefs" "${INTERSHEET_REFS}" (at 133.35 89.84 90)
+      (effects (font (size 1.27 1.27)) (justify right) hide)
+    )
+  )
   (global_label "12" (shape input) (at 49.53 119.38 180) (fields_autoplaced)
     (effects (font (size 1.27 1.27)) (justify right))
@@
     )
   )
+  (global_label "17" (shape input) (at 158.75 72.39 270) (fields_autoplaced)
+    (effects (font (size 1.27 1.27)) (justify right))
+    (property "Intersheetrefs" "${INTERSHEET_REFS}" (at 158.75 77.14 90)
+      (effects (font (size 1.27 1.27)) (justify right) hide)
+    )
+  )
+  (global_label "18" (shape input) (at 156.21 72.39 270) (fields_autoplaced)
+    (effects (font (size 1.27 1.27)) (justify right))
+    (property "Intersheetrefs" "${INTERSHEET_REFS}" (at 156.21 77.14 90)
+      (effects (font (size 1.27 1.27)) (justify right) hide)
+    )
+  )
   (global_label "0" (shape input) (at 44.45 34.29 180) (fields_autoplaced)
     (effects (font (size 1.27 1.27)) (justify right))
@@
     )
   )
+  (global_label "GND" (shape input) (at 143.51 85.09 270) (fields_autoplaced)
+    (effects (font (size 1.27 1.27)) (justify right))
+    (property "Intersheetrefs" "${INTERSHEET_REFS}" (at 143.51 91.2915 90)
+      (effects (font (size 1.27 1.27)) (justify right) hide)
+    )
+  )
   (global_label "8" (shape input) (at 49.53 106.68 180) (fields_autoplaced)
     (effects (font (size 1.27 1.27)) (justify right))
@@
     )
   )
+  (global_label "5" (shape input) (at 118.11 85.09 270) (fields_autoplaced)
+    (effects (font (size 1.27 1.27)) (justify right))
+    (property "Intersheetrefs" "${INTERSHEET_REFS}" (at 118.11 88.6305 90)
+      (effects (font (size 1.27 1.27)) (justify right) hide)
+    )
+  )
+  (global_label "7" (shape input) (at 118.11 62.23 270) (fields_autoplaced)
+    (effects (font (size 1.27 1.27)) (justify right))
+    (property "Intersheetrefs" "${INTERSHEET_REFS}" (at 118.11 65.7705 90)
+      (effects (font (size 1.27 1.27)) (justify right) hide)
+    )
+  )
   (global_label "GND" (shape input) (at 85.09 124.46 0) (fields_autoplaced)
     (effects (font (size 1.27 1.27)) (justify left))
@@
     (property "Intersheetrefs" "${INTERSHEET_REFS}" (at 92.0172 83.82 0)
       (effects (font (size 1.27 1.27)) (justify left) hide)
+    )
+  )
+  (global_label "10" (shape input) (at 133.35 62.23 270) (fields_autoplaced)
+    (effects (font (size 1.27 1.27)) (justify right))
+    (property "Intersheetrefs" "${INTERSHEET_REFS}" (at 133.35 66.98 90)
+      (effects (font (size 1.27 1.27)) (justify right) hide)
     )
   )
@@
       (effects (font (size 1.27 1.27)))
     )
-    (property "Footprint" "TypeC:HRO_TYPE-C-31-M-12" (at 69.85 39.37 0)
+    (property "Footprint" "USB-C-Power-tester:TYPE-C-31-M-12" (at 69.85 39.37 0)
       (effects (font (size 1.27 1.27)) (justify bottom) hide)
     )
