File: Kicad/Keeb_small_symetrical_hotswap_left/Keeb.kicad_sch (KiCad schematic)
At the start: 20 parts, among them J1 TYPE-C-31-M-12, SW1 CherryMX, SW10 CherryMX, SW11 CherryMX, SW13 CherryMX, SW14 CherryMX, SW15 CherryMX, SW16 CherryMX, SW17 CherryMX, SW18 CherryMX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

Commit message: rm holes for controller
Parts:
- U1: footprint MCU_RaspberryPi_and_Boards:RPi_Pico_SMD_TH -> MCU_RaspberryPi_and_Boards:RPi_Pico_SMD_TH_NO_HOLES
Changed lines of the file:
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@@
       (effects (font (size 1.27 1.27)))
     )
-    (property "Footprint" "MCU_RaspberryPi_and_Boards:RPi_Pico_SMD_TH" (at 67.31 105.41 90)
+    (property "Footprint" "MCU_RaspberryPi_and_Boards:RPi_Pico_SMD_TH_NO_HOLES" (at 67.31 105.41 90)
       (effects (font (size 1.27 1.27)) hide)
     )

Commit message: min
Parts:
- J1: footprint USB-C-Power-tester:TYPE-C-31-M-12 -> TypeC:HRO_TYPE-C-31-M-12
Changed lines of the file:
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@@
       (effects (font (size 1.27 1.27)))
     )
-    (property "Footprint" "USB-C-Power-tester:TYPE-C-31-M-12" (at 69.85 39.37 0)
+    (property "Footprint" "TypeC:HRO_TYPE-C-31-M-12" (at 69.85 39.37 0)
       (effects (font (size 1.27 1.27)) (justify bottom) hide)
     )

Commit message: Added mounting holes to the PCB
Parts:
- added H1, H2, H3, H4, H5, H7, H8, H9: MountingHole, MountingHole:MountingHole_3.2mm_M3, symbol Mechanical:MountingHole
Changed lines of the file:
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@@
+    )
+  )
+  (symbol (lib_id "Mechanical:MountingHole") (at 191.77 22.86 0) (unit 1)
+    (in_bom yes) (on_board yes) (dnp no) (fields_autoplaced)
+    (property "Reference" "H7" (at 194.31 21.59 0)
+      (effects (font (size 1.27 1.27)) (justify left))
+    )
+    (property "Value" "MountingHole" (at 194.31 24.13 0)
+      (effects (font (size 1.27 1.27)) (justify left))
+    )
+    (property "Footprint" "MountingHole:MountingHole_3.2mm_M3" (at 191.77 22.86 0)
+      (effects (font (size 1.27 1.27)) hide)
+    )
+    (property "Datasheet" "~" (at 191.77 22.86 0)
+      (effects (font (size 1.27 1.27)) hide)
+    )
+    (instances
+      (project "Keeb"
+        (path "/f8892ba2-997e-41dc-a7e4-c2b6962ff100"
+          (reference "H7") (unit 1)
+        )
+      )
     )
   )
@@
         )
       )
+    )
+  )
+  (symbol (lib_id "Mechanical:MountingHole") (at 191.77 26.67 0) (unit 1)
+    (in_bom yes) (on_board yes) (dnp no) (fields_autoplaced)
+    (property "Reference" "H8" (at 194.31 25.4 0)
+      (effects (font (size 1.27 1.27)) (justify left))
+    )
+    (property "Value" "MountingHole" (at 194.31 27.94 0)
+      (effects (font (size 1.27 1.27)) (justify left))
+    )
+    (property "Footprint" "MountingHole:MountingHole_3.2mm_M3" (at 191.77 26.67 0)
+      (effects (font (size 1.27 1.27)) hide)
+    )
+    (property "Datasheet" "~" (at 191.77 26.67 0)
+      (effects (font (size 1.27 1.27)) hide)
+    )
+    (instances
+      (project "Keeb"
+        (path "/f8892ba2-997e-41dc-a7e4-c2b6962ff100"
+          (reference "H8") (unit 1)
+        )
+      )
+    )
+  )
+  (symbol (lib_id "Mechanical:MountingHole") (at 175.26 22.86 0) (unit 1)
+    (in_bom yes) (on_board yes) (dnp no) (fields_autoplaced)
+    (property "Reference" "H4" (at 177.8 21.59 0)
+      (effects (font (size 1.27 1.27)) (justify left))
+    )
+    (property "Value" "MountingHole" (at 177.8 24.13 0)
+      (effects (font (size 1.27 1.27)) (justify left))
+    )
+    (property "Footprint" "MountingHole:MountingHole_3.2mm_M3" (at 175.26 22.86 0)
+      (effects (font (size 1.27 1.27)) hide)
+    )
+    (property "Datasheet" "~" (at 175.26 22.86 0)
+      (effects (font (size 1.27 1.27)) hide)
+    )
+    (instances
+      (project "Keeb"
+        (path "/f8892ba2-997e-41dc-a7e4-c2b6962ff100"
+          (reference "H4") (unit 1)
+        )
+      )
+    )
+  )
+  (symbol (lib_id "Mechanical:MountingHole") (at 156.21 22.86 0) (unit 1)
+    (in_bom yes) (on_board yes) (dnp no) (fields_autoplaced)
+    (property "Reference" "H1" (at 158.75 21.59 0)
+      (effects (font (size 1.27 1.27)) (justify left))
+    )
+    (property "Value" "MountingHole" (at 158.75 24.13 0)
+      (effects (font (size 1.27 1.27)) (justify left))
+    )
+    (property "Footprint" "MountingHole:MountingHole_3.2mm_M3" (at 156.21 22.86 0)
+      (effects (font (size 1.27 1.27)) hide)
+    )
+    (property "Datasheet" "~" (at 156.21 22.86 0)
+      (effects (font (size 1.27 1.27)) hide)
+    )
+    (instances
+      (project "Keeb"
+        (path "/f8892ba2-997e-41dc-a7e4-c2b6962ff100"
+          (reference "H1") (unit 1)
+        )
+      )
+    )
+  )
+  (symbol (lib_id "Mechanical:MountingHole") (at 156.21 27.94 0) (unit 1)
+    (in_bom yes) (on_board yes) (dnp no) (fields_autoplaced)
+    (property "Reference" "H2" (at 158.75 26.67 0)
+      (effects (font (size 1.27 1.27)) (justify left))
+    )
+    (property "Value" "MountingHole" (at 158.75 29.21 0)
+      (effects (font (size 1.27 1.27)) (justify left))
+    )
+    (property "Footprint" "MountingHole:MountingHole_3.2mm_M3" (at 156.21 27.94 0)
+      (effects (font (size 1.27 1.27)) hide)
+    )
+    (property "Datasheet" "~" (at 156.21 27.94 0)
+      (effects (font (size 1.27 1.27)) hide)
+    )
+    (instances
+      (project "Keeb"
+        (path "/f8892ba2-997e-41dc-a7e4-c2b6962ff100"
+          (reference "H2") (unit 1)
+        )
+      )
+    )
+  )
+  (symbol (lib_id "Mechanical:MountingHole") (at 156.21 33.02 0) (unit 1)
+    (in_bom yes) (on_board yes) (dnp no) (fields_autoplaced)
+    (property "Reference" "H3" (at 158.75 31.75 0)
+      (effects (font (size 1.27 1.27)) (justify left))
+    )
+    (property "Value" "MountingHole" (at 158.75 34.29 0)
+      (effects (font (size 1.27 1.27)) (justify left))
+    )
+    (property "Footprint" "MountingHole:MountingHole_3.2mm_M3" (at 156.21 33.02 0)
+      (effects (font (size 1.27 1.27)) hide)
+    )
+    (property "Datasheet" "~" (at 156.21 33.02 0)
+      (effects (font (size 1.27 1.27)) hide)
+    )
+    (instances
+      (project "Keeb"
+        (path "/f8892ba2-997e-41dc-a7e4-c2b6962ff100"
+          (reference "H3") (unit 1)
+        )
+      )
+    )
+  )
+  (symbol (lib_id "Mechanical:MountingHole") (at 175.26 27.94 0) (unit 1)
+    (in_bom yes) (on_board yes) (dnp no) (fields_autoplaced)
+    (property "Reference" "H5" (at 177.8 26.67 0)
+      (effects (font (size 1.27 1.27)) (justify left))
+    )
+    (property "Value" "MountingHole" (at 177.8 29.21 0)
+      (effects (font (size 1.27 1.27)) (justify left))
+    )
+    (property "Footprint" "MountingHole:MountingHole_3.2mm_M3" (at 175.26 27.94 0)
+      (effects (font (size 1.27 1.27)) hide)
+    )
+    (property "Datasheet" "~" (at 175.26 27.94 0)
+      (effects (font (size 1.27 1.27)) hide)
+    )
+    (instances
+      (project "Keeb"
+        (path "/f8892ba2-997e-41dc-a7e4-c2b6962ff100"
+          (reference "H5") (unit 1)
+        )
+      )
+    )
+  )
+  (symbol (lib_id "Mechanical:MountingHole") (at 191.77 30.48 0) (unit 1)
+    (in_bom yes) (on_board yes) (dnp no) (fields_autoplaced)
+    (property "Reference" "H9" (at 194.31 29.21 0)
+      (effects (font (size 1.27 1.27)) (justify left))
+    )
+    (property "Value" "MountingHole" (at 194.31 31.75 0)
+      (effects (font (size 1.27 1.27)) (justify left))
+    )
+    (property "Footprint" "MountingHole:MountingHole_3.2mm_M3" (at 191.77 30.48 0)
+      (effects (font (size 1.27 1.27)) hide)
+    )
+    (property "Datasheet" "~" (at 191.77 30.48 0)
+      (effects (font (size 1.27 1.27)) hide)
+    )
+    (instances
+      (project "Keeb"
+        (path "/f8892ba2-997e-41dc-a7e4-c2b6962ff100"
+          (reference "H9") (unit 1)
+        )
+      )
